File: io/vcafd_io.kicad_pcb (KiCad board)
At the start: 2 copper layers, 40.5 x 100 mm, 37 parts, among them J1 AudioJack2_SwitchT, J2 AudioJack2_SwitchT, J3 AudioJack2_SwitchT, J4 AudioJack2_SwitchT, J5 AudioJack2_SwitchT, J6 AudioJack2_SwitchT, J7 Conn_01x09_Pin, J8 Conn_01x09_Pin, J9 Conn_01x09_Pin, Q1 2N7002, Q2 2N7002, Q3 2N7002, Q4 2N7002, SW1 SW_SPDT, SW2 SW_SPDT

Commit message: Connect CV Tn to ground
Connections:
- J3 pad TN: unconnected-(J3-PadTN) -> GND
