File: core/agc.kicad_sch (KiCad schematic)
At the start: 29 parts, among them Q17 MMBT3904, Q18 MMBT3906, Q19 MMBFJ113, Q20 MMBT3906, Q21 MMBT3904, Q22 MMBT3906, Q23 MMBT3906, Q24 BSS84, Q25 MMBT3904, Q26 MMBT3906, U11 TL072

Commit message: Update partnames
Parts:
- R92: now not fitted
Changed lines of the file:
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@@
 		(in_bom yes)
 		(on_board yes)
-		(dnp no)
+		(dnp yes)
 		(fields_autoplaced yes)
 		(property "Reference" "R92"

Commit message: Fixes for v1.1
Parts:
- C24: renamed from C22; now not fitted
- renumbered C21 to C23, C23 to C25, C24 to C26, C25 to C27, Q17 to Q19, Q18 to Q20, Q19 to Q21, Q20 to Q22, Q21 to Q23, Q22 to Q24, Q23 to Q25, Q24 to Q26, Q25 to Q27, Q26 to Q28, R91 to R83, R92 to R84, R93 to R85, R94 to R86, R95 to R87, R96 to R88, R97 to R89, R98 to R90, R99 to R91, R100 to R92, R101 to R93, R102 to R94, R103 to R95
