File: core/vcafd.kicad_pcb (KiCad board)
At the start: 4 copper layers, 40.5 x 100 mm, 225 parts, among them J1 Conn_02x08_Odd_Even, J2 Conn_01x09_Socket, J3 Conn_01x09_Socket, J4 Conn_01x09_Socket, Q1 ZXMP3A13FTA, Q10 MMBT3906, Q11 BSS84, Q12 MMBT3904, Q13 MMBT3904, Q14 MMBT3906, Q15 MMBT3906, Q16 MMBT3904, Q17 MMBT3904, Q18 MMBT3906, Q19 MMBFJ113, Q2 PMV88ENER, Q20 MMBT3906, Q21 MMBT3904, Q22 MMBT3906, Q23 MMBT3906, Q24 BSS84, Q25 MMBT3904, Q26 MMBT3906, Q3 BSS84, Q4 MMBT3904, Q5 MMBT3904, Q6 MMBT3906, Q7 MMBT3906, Q8 MMBT3904, Q9 MMBT3906, U1 TL072, U10 TL072, U11 TL072, U2 TL072, U3 TL072, U4 TL072, U5 LM13700, U6 TL072, U7 TL072, U8 TL072, U9 TL072

Commit message: Gerbers setup
Parts:
- R11, R61: value 5k1 -> 15k
- R18, R19: value ??? -> 8k2
- R39, R40: value 13k -> 12k
- R41, R42: value 30k -> 39k
- R58, R90: value 1M -> 1M5
Changed lines of the file:
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@@
 			(plot_on_all_layers_selection 0x0000000_00000000)
 			(disableapertmacros no)
-			(usegerberextensions no)
-			(usegerberattributes yes)
-			(usegerberadvancedattributes yes)
-			(creategerberjobfile yes)
+			(usegerberextensions yes)
+			(usegerberattributes no)
+			(usegerberadvancedattributes no)
+			(creategerberjobfile no)
 			(dashed_line_dash_ratio 12.000000)
 			(dashed_line_gap_ratio 3.000000)
@@
 			(psa4output no)
 			(plotreference yes)
-			(plotvalue yes)
+			(plotvalue no)
 			(plotfptext yes)
 			(plotinvisibletext no)
 			(sketchpadsonfab no)
-			(subtractmaskfromsilk no)
+			(subtractmaskfromsilk yes)
 			(outputformat 1)
 			(mirror no)
-			(drillshape 1)
+			(drillshape 0)
 			(scaleselection 1)
-			(outputdirectory "")
+			(outputdirectory "out/")
 		)
 	)
@@
 			)
 		)
-		(property "Value" "5k1"
+		(property "Value" "15k"
 			(at 0 1.43 0)
 			(layer "F.Fab")
@@
 			)
 		)
-		(property "Value" "???"
+		(property "Value" "8k2"
 			(at 0 1.43 0)
 			(layer "F.Fab")
@@
 			)
 		)
-		(property "Value" "5k1"
+		(property "Value" "15k"
 			(at 0 1.43 0)
 			(layer "F.Fab")
@@
 			)
 		)
-		(property "Value" "???"
+		(property "Value" "8k2"
 			(at 0 1.43 0)
 			(layer "F.Fab")
@@
 			)
 		)
-		(property "Value" "13k"
+		(property "Value" "12k"
 			(at 0 1.43 0)
 			(layer "F.Fab")
@@
 			)
 		)
-		(property "Value" "13k"
+		(property "Value" "12k"
 			(at 0 1.43 0)
 			(layer "F.Fab")
@@
 			)
 		)
-		(property "Value" "30k"
+		(property "Value" "39k"
 			(at 0 -1.43 90)
 			(layer "B.Fab")
@@
 			)
 		)
-		(property "Value" "30k"
+		(property "Value" "39k"
 			(at 0 -1.43 90)
 			(layer "B.Fab")
@@
 			)
 		)
-		(property "Value" "1M"
+		(property "Value" "1M5"
 			(at 0 -1.43 0)
 			(layer "B.Fab")
@@
 			)
 		)
-		(property "Value" "1M"
+		(property "Value" "1M5"
 			(at 0 -1.43 0)
 			(layer "B.Fab")

Commit message: Fixes for v1.1
Parts:
- removed the D37 at (164.0, 54.0)
- removed the D38 at (159.5, 54.0)
- removed the D5 at (180.5, 54.0)
- removed the D6 at (176.0, 54.0)
- removed the Q11 at (167.5, 61.5)
- removed the Q3 at (184.0, 61.5)
- removed the R11 at (180.5, 63.0)
- removed the R61 at (164.0, 63.0)
- added C15: 470n C0G, Capacitor_SMD:C_1206_3216Metric, B.Cu at (181.2, 78.8)
- added C22: 470n C0G, Capacitor_SMD:C_1206_3216Metric, B.Cu at (175.8, 78.8)
- added Q17: MMBT3906, Package_TO_SOT_SMD:SOT-23, F.Cu at (163.6, 53.4)
- added Q18: MMBT3904, Package_TO_SOT_SMD:SOT-23, F.Cu at (158.6, 53.4)
- added Q8: MMBT3906, Package_TO_SOT_SMD:SOT-23, F.Cu at (180.0, 53.4)
- added Q9: MMBT3904, Package_TO_SOT_SMD:SOT-23, F.Cu at (175.2, 53.4)
- D1, D2, D3, D4: value D -> 1N4148
- D10: renamed from D12; value D -> 1N4148
- D11: renamed from D13; value D -> 1N4148
- D12: renamed from D14; value D -> 1N4148
- D13: renamed from D15; value D -> 1N4148
- D14: renamed from D16; value D -> 1N4148
- D15: renamed from D17; value D -> 1N4148
- D16: renamed from D18; value D -> 1N4148
- D17: renamed from D19; value D -> 1N4148
- D18: renamed from D20; value D -> 1N4148
- D19: renamed from D21; value D -> 1N4148
- D20: renamed from D22; value D -> 1N4148
- D21: renamed from D23; value D -> 1N4148
- D22: renamed from D24; value D -> 1N4148
- D23: renamed from D25; value D -> 1N4148
- D24: renamed from D26; value D -> 1N4148
- D25: renamed from D27; value D -> 1N4148
- D26: renamed from D28; value D -> 1N4148
- D27: renamed from D29; value D -> 1N4148
- D28: renamed from D30; value D -> 1N4148
- D29: renamed from D31; value D -> 1N4148
- D30: renamed from D32; value D -> 1N4148
- D31: renamed from D33; value D -> 1N4148
- D32: renamed from D34; value D -> 1N4148
- D33: renamed from D35; value D -> 1N4148
- D34: renamed from D36; value D -> 1N4148
- D35: renamed from D39; value D -> 1N4148
- D36: renamed from D40; value D -> 1N4148
- D37: renamed from D41; value D -> 1N4148
- D38: renamed from D42; value D -> 1N4148
- D39: renamed from D43; value D -> 1N4148
- D40: renamed from D44; value D -> 1N4148
- D41: renamed from D45; value D -> 1N4148
- D42: renamed from D46; value D -> 1N4148
- D43: renamed from D47; value D -> 1N4148
- D44: renamed from D48; value D -> 1N4148
- D45: renamed from D49; value D -> 1N4148
- D46: renamed from D50; value D -> 1N4148
- D47: renamed from D51; value D -> 1N4148
- D48: renamed from D52; value D -> 1N4148
- D49: renamed from D53; value D -> 1N4148
- D5: renamed from D7; value D -> 1N4148
- D50: renamed from D54; value D -> 1N4148
- D51: renamed from D55; value D -> 1N4148
- D52: renamed from D56; value D -> 1N4148
- D53: renamed from D57; value D -> 1N4148
- D54: renamed from D58; value D -> 1N4148
- D55: renamed from D59; value D -> 1N4148
- D56: renamed from D60; value D -> 1N4148
- D57: renamed from D61; value D -> 1N4148
- D58: renamed from D62; value D -> 1N4148
- D6: renamed from D8; value D -> 1N4148
- D7: renamed from D9; value D -> 1N4148
- D8: renamed from D10; value D -> 1N4148
- D9: renamed from D11; value D -> 1N4148
- Q1: value ZXMP3A13FTA -> DMP3099
- Q2: value PMV88ENER -> DMN6075
- R12: renamed from R18; value 8k2 -> 4k3
- R18: renamed from R22; value 3k3 -> 2k
- R19: renamed from R23; value 15k -> 18k
- R26: renamed from R30; value 100k -> 47k
- R28: renamed from R32; value 100k -> 47k
- R35: renamed from R39; value 12k -> 39k
- R36: renamed from R40; value 12k -> 39k
- R37: renamed from R41; value 39k -> 51k
- R38: renamed from R42; value 39k -> 51k
- R45: renamed from R49; value 100 -> 200
- R58: renamed from R19; value 8k2 -> 4k3
- R64: renamed from R72; value 3k3 -> 2k
- R65: renamed from R73; value 15k -> 18k
- R73: renamed from R81; value 100 -> 200
- moved C1 12.1 mm to (176.0, 125.0), turned to 0 degrees
- moved C2 12.1 mm to (165.0, 120.0), turned to 0 degrees
- renumbered C15 to C16, C16 to C17, C17 to C18, C18 to C19, C19 to C20, C20 to C21, C21 to C23, C22 to C24, C23 to C25, C24 to C26, C25 to C27, Q9 to Q10, Q10 to Q11, Q17 to Q19, Q18 to Q20, Q19 to Q21, Q20 to Q22, Q21 to Q23, Q22 to Q24, Q23 to Q25, Q24 to Q26, Q25 to Q27, Q26 to Q28, Q4 to Q3, Q5 to Q4, Q6 to Q5, Q7 to Q6, Q8 to Q7, R13 to R10, R10 to R11, R12 to R13, R24 to R20, R25 to R21, R26 to R22, R27 to R23, R28 to R24, R29 to R25, R31 to R27, R33 to R29, R34 to R30, R35 to R31, R36 to R32, R37 to R33, R38 to R34, R43 to R39, R44 to R40, R45 to R41, R46 to R42, R47 to R43, R48 to R44, R50 to R46, R51 to R47, R52 to R48, R53 to R49, R54 to R50, R55 to R51, R56 to R52, R57 to R53, R58 to R54, R59 to R55, R63 to R56, R60 to R57, R62 to R59, R64 to R60, R65 to R61, R66 to R62, R67 to R63, R74 to R66, R75 to R67, R76 to R68, R77 to R69, R78 to R70, R79 to R71, R80 to R72, R82 to R74, R83 to R75, R84 to R76, R85 to R77, R86 to R78, R87 to R79, R88 to R80, R89 to R81, R90 to R82, R91 to R83, R92 to R84, R93 to R85, R94 to R86, R95 to R87, R96 to R88, R97 to R89, R98 to R90, R99 to R91, R100 to R92, R101 to R93, R102 to R94, R103 to R95
Connections:
- Q6 pad 2: Net-(Q7-E) -> Net-(Q6-E)
- Q7 pad 2: Net-(Q7-E) -> Net-(Q6-E)
- R14 pad 2: Net-(Q7-E) -> Net-(Q6-E)
- R18 pad 1: Net-(Q7-E) -> Net-(R18-Pad1)
- R18 pad 2: Net-(D5-A) -> Net-(Q6-E)
- R19 pad 1: Net-(D5-A) -> Net-(Q6-E)
- R54 pad 2: Fold_A -> Net-(C15-Pad1)
- R64 pad 1: Net-(Q15-E) -> Net-(R64-Pad1)
- R64 pad 2: Net-(D37-A) (its old number) -> Net-(Q15-E)
- R65 pad 1: Net-(D37-A) (its old number) -> Net-(Q15-E)
- R82 pad 2: Fold_B -> Net-(C22-Pad1)
- U1 pad 4: +VDC -> -VDC
- U1 pad 8: -VDC -> +VDC
- U10 pad 7: Fold_B -> Net-(C22-Pad1)
- U4 pad 1: Net-(Q7-E) -> Net-(R18-Pad1)
- U7 pad 7: Fold_A -> Net-(C15-Pad1)
- U9 pad 1: Net-(Q15-E) -> Net-(R64-Pad1)
Routing:
- net Net-(Q6-E): track 0.00 -> 36.3 mm, vias 0 -> 1
- net Net-(Q15-E): track 17.7 -> 36.6 mm, vias 0 -> 1
- net Net-(Q7-E): track 17.4 -> 0.00 mm
- net Net-(D5-A): track 12.8 -> 0.00 mm, vias 1 -> 0
- net Net-(D37-A) (its old number): track 12.8 -> 0.00 mm, vias 1 -> 0
- net -VDC: track 71.0 -> 78.1 mm, vias 14 -> 16
- net Net-(C15-Pad1): track 0.00 -> 6.31 mm
- net Fold_B: track 20.1 -> 15.5 mm
- net Fold_A: track 45.1 -> 40.6 mm
- net Net-(C22-Pad1): track 0.00 -> 4.12 mm
- net Net-(U3B-+): track 7.37 -> 4.07 mm
- net +VDC: track 76.5 -> 79.8 mm, vias 14 -> 16
- net Net-(U8B-+): track 7.23 -> 4.07 mm
- net Net-(Q11-D): track 2.45 -> 0.00 mm
- net Net-(Q3-D): track 2.36 -> 0.00 mm
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Other:
- board text added: "ACID VCA Core v1.1"
- board text removed: "ACID VCA Core v1.0"
