File: core/vcafd.kicad_sch (KiCad schematic)
At the start: 20 parts, among them J1 Conn_02x08_Odd_Even, J2 Conn_01x09_Socket, J3 Conn_01x09_Socket, J4 Conn_01x09_Socket, Q1 ZXMP3A13FTA, Q2 PMV88ENER, U1 TL072, U2 TL072

Commit message: Update partnames
Parts:
- Q1: value ZXMP3A13FTA -> DMP3099
- Q2: value PMV88ENER -> DMN6075
Changed lines of the file:
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@@
 			)
 		)
-		(property "Value" "PMV88ENER"
+		(property "Value" "DMN6075"
 			(at 63.5 194.31 90)
 			(effects
@@
 			)
 		)
-		(property "Value" "ZXMP3A13FTA"
+		(property "Value" "DMP3099"
 			(at 63.5 151.13 90)
 			(effects

Commit message: Fixes for v1.1
Connections:
- net +VDC: now also U1.8 (V+); no longer U1.4 (V-)
- net -VDC: now also U1.4 (V-); no longer U1.8 (V+)
Changed lines of the file:
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@@
 (kicad_sch
-	(version 20231120)
+	(version 20250114)
 	(generator "eeschema")
-	(generator_version "8.0")
+	(generator_version "9.0")
 	(paper "A4")
 	(title_block
 		(title "ACID VCA CORE")
-		(date "2025-03-27")
-		(rev "1.0")
+		(date "2025-05-18")
+		(rev "1.1")
+	)
+	(text "The AGC can be removed, but U2 should be non-inverting in that case.\nDoing that would mean the output amplitude is halved when one channel is quiet"
+		(exclude_from_sim no)
+		(at 230.886 98.044 0)
+		(effects
+			(font
+				(size 1.27 1.27)
+			)
+		)
 	)
 	(junction
@@
 		)
 	)
-	(text "The AGC can be removed, but U2 should be non-inverting in that case.\nDoing that would mean the output amplitude is halved when one channel is quiet"
-		(exclude_from_sim no)
-		(at 230.886 98.044 0)
-		(effects
-			(font
-				(size 1.27 1.27)
-			)
-		)
-	)
 	(global_label "Offset_B"
 		(shape output)
@@
 		(dnp no)
 		(fields_autoplaced yes)
-		(property "Reference" "#PWR09"
+		(property "Reference" "#PWR010"
 			(at 111.76 125.73 0)
 			(effects
@@
 			(project ""
 				(path "/dc073820-51c1-4a11-816f-0331d71182e9"
-					(reference "#PWR09")
+					(reference "#PWR010")
 					(unit 1)
 				)
@@
 		(lib_id "Amplifier_Operational:TL072")
 		(at 111.76 172.72 0)
-		(mirror x)
 		(unit 3)
 		(exclude_from_sim no)
@@
 		(on_board yes)
 		(dnp no)
-		(fields_autoplaced yes)
 		(property "Reference" "U1"
-			(at 107.95 171.4499 0)
+			(at 107.95 173.9901 0)
 			(effects
 				(font
@@
 		)
 		(property "Value" "TL072"
-			(at 107.95 173.9899 0)
+			(at 107.95 171.4501 0)
 			(effects
 				(font
@@
 		(dnp no)
 		(fields_autoplaced yes)
-		(property "Reference" "#PWR010"
+		(property "Reference" "#PWR09"
 			(at 111.76 115.57 0)
 			(effects
@@
 			(project ""
 				(path "/dc073820-51c1-4a11-816f-0331d71182e9"
-					(reference "#PWR010")
+					(reference "#PWR09")
 					(unit 1)
 				)
@@
 		(at 172.72 50.8)
 		(size 15.24 15.24)
+		(exclude_from_sim no)
+		(in_bom yes)
+		(on_board yes)
+		(dnp no)
 		(fields_autoplaced yes)
 		(stroke
@@
 		(at 172.72 25.4)
 		(size 15.24 15.24)
+		(exclude_from_sim no)
+		(in_bom yes)
+		(on_board yes)
+		(dnp no)
 		(fields_autoplaced yes)
 		(stroke
@@
 		(at 82.55 43.18)
 		(size 16.51 22.86)
+		(exclude_from_sim no)
+		(in_bom yes)
+		(on_board yes)
+		(dnp no)
 		(fields_autoplaced yes)
 		(stroke
@@
 		(at 121.92 49.53)
 		(size 15.24 15.24)
+		(exclude_from_sim no)
+		(in_bom yes)
+		(on_board yes)
+		(dnp no)
 		(fields_autoplaced yes)
 		(stroke
@@
 		(at 121.92 24.13)
 		(size 15.24 15.24)
+		(exclude_from_sim no)
+		(in_bom yes)
+		(on_board yes)
+		(dnp no)
 		(fields_autoplaced yes)
 		(stroke
@@
 		(at 215.9 76.2)
 		(size 20.32 11.43)
+		(exclude_from_sim no)
+		(in_bom yes)
+		(on_board yes)
+		(dnp no)
 		(fields_autoplaced yes)
 		(stroke
@@
 		)
 	)
+	(embedded_fonts no)
 )
